File: Hardware/3DoT-Hexy-Shield.sch (EAGLE design)
At the start: 0 parts

Commit message: Finished board layout for the shield
Parts:
- added JP1, JP2: (no value), pinhead:PINHD-1X8
- added JP3, JP4: (no value), pinhead:PINHD-1X4
- added JP5, JP6: (no value), pinhead:PINHD-1X3
- added RESET: (no value), SparkFun-Switches:MOMENTARY-SWITCH-SPST-2-SMD-5.2MM
Connections:
- new net 3.3V: JP2.6, JP3.1, JP4.1, JP5.1, JP6.1
- new net 5V: JP1.7
- new net A4: JP1.6
- new net AREF: JP1.5
- new net GND: JP2.7, JP3.4, JP4.4, JP5.2, JP6.2, RESET.3, RESET.4
- new net MISO: JP1.1, JP4.2
- new net MOSI: JP1.2, JP4.3
- new net RAW: JP1.8
- new net RESET: JP2.1, RESET.1, RESET.2
- new net RXI1: JP2.4
- new net SCK: JP1.3, JP3.2
- new net SCL: JP2.2, JP5.3
- new net SDA: JP2.3, JP6.3
- new net SS: JP1.4, JP3.3
- new net TXO1: JP2.5
- new net VM: JP2.8
Other:
- note added: "D14 (PCINT3)"
- note added: "D15 (PCINT1)"
- note added: "D16 (PCINT2)"
- note added: "D17/RX LED (PCINT0)"
- note added: "D2 (INT1)"
- note added: "D3# (INT0)"
